Commit message: getting there :)

File: apps/models/urdf/phantomx.urdf (robot description, URDF)
Before this commit: robot PhantomX, 26 links, 25 joints
Links:
- link MP_BODY: geometry collision mesh filename=meshes/body_coll.STL scale=1 1 1; visual mesh filename=meshes/body.STL scale=1 1 1
- link c1_lf: geometry collision mesh filename=meshes/connect_coll.STL scale=1 1 1; visual mesh filename=meshes/connect.STL scale=1 1 1
- link c1_lm: geometry collision mesh filename=meshes/connect_coll.STL scale=1 1 1; visual mesh filename=meshes/connect.STL scale=1 1 1
- link c1_lr: geometry collision mesh filename=meshes/connect_coll.STL scale=1 1 1; visual mesh filename=meshes/connect.STL scale=1 1 1
- link c1_rf: geometry collision mesh filename=meshes/connect_coll.STL scale=1 1 1; visual mesh filename=meshes/connect.STL scale=1 1 1
- link c1_rm: geometry collision mesh filename=meshes/connect_coll.STL scale=1 1 1; visual mesh filename=meshes/connect.STL scale=1 1 1
- link c1_rr: geometry collision mesh filename=meshes/connect_coll.STL scale=1 1 1; visual mesh filename=meshes/connect.STL scale=1 1 1
- link c2_lf: geometry collision mesh filename=meshes/connect_coll.STL scale=1 1 1; visual mesh filename=meshes/connect.STL scale=1 1 1
- link c2_lm: geometry collision mesh filename=meshes/connect_coll.STL scale=1 1 1; visual mesh filename=meshes/connect.STL scale=1 1 1
- link c2_lr: geometry collision mesh filename=meshes/connect_coll.STL scale=1 1 1; visual mesh filename=meshes/connect.STL scale=1 1 1
- link c2_rf: geometry collision mesh filename=meshes/connect_coll.STL scale=1 1 1; visual mesh filename=meshes/connect.STL scale=1 1 1
- link c2_rm: geometry collision mesh filename=meshes/connect_coll.STL scale=1 1 1; visual mesh filename=meshes/connect.STL scale=1 1 1
- link c2_rr: geometry collision mesh filename=meshes/connect_coll.STL scale=1 1 1; visual mesh filename=meshes/connect.STL scale=1 1 1
- link thigh_lf: geometry collision mesh filename=meshes/thigh_l_coll.STL scale=1 1 1; visual mesh filename=meshes/thigh_l.STL scale=1 1 1
- link thigh_lm: geometry collision mesh filename=meshes/thigh_l_coll.STL scale=1 1 1; visual mesh filename=meshes/thigh_l.STL scale=1 1 1
- link thigh_lr: geometry collision mesh filename=meshes/thigh_l_coll.STL scale=1 1 1; visual mesh filename=meshes/thigh_l.STL scale=1 1 1
- link thigh_rf: geometry collision mesh filename=meshes/thigh_l_coll.STL scale=1 1 1; visual mesh filename=meshes/thigh_l.STL scale=1 1 1
- link thigh_rm: geometry collision mesh filename=meshes/thigh_l_coll.STL scale=1 1 1; visual mesh filename=meshes/thigh_l.STL scale=1 1 1
- link thigh_rr: geometry collision mesh filename=meshes/thigh_l_coll.STL scale=1 1 1; visual mesh filename=meshes/thigh_l.STL scale=1 1 1
- link tibia_lf: geometry collision mesh filename=meshes/tibia_l_coll.STL scale=1 1 1; visual mesh filename=meshes/tibia_l.STL scale=1 1 1
- link tibia_lm: geometry collision mesh filename=meshes/tibia_l_coll.STL scale=1 1 1; visual mesh filename=meshes/tibia_l.STL scale=1 1 1
- link tibia_lr: geometry collision mesh filename=meshes/tibia_l_coll.STL scale=1 1 1; visual mesh filename=meshes/tibia_l.STL scale=1 1 1
- link tibia_rf: geometry collision mesh filename=meshes/tibia_l_coll.STL scale=1 1 1; visual mesh filename=meshes/tibia_l.STL scale=1 1 1
- link tibia_rm: geometry collision mesh filename=meshes/tibia_l_coll.STL scale=1 1 1; visual mesh filename=meshes/tibia_l.STL scale=1 1 1
- link tibia_rr: geometry collision mesh filename=meshes/tibia_l_coll.STL scale=1 1 1; visual mesh filename=meshes/tibia_l.STL scale=1 1 1

Commit message: models load(yay).. visual links needs to be in objs not stls

File: apps/models/urdf/phantomx.urdf (robot description, URDF)
Before this commit: robot PhantomX, 26 links, 25 joints
Links:
- link MP_BODY: geometry collision mesh filename=../meshes/body_coll.STL scale=1 1 1; visual mesh filename=../meshes/body.STL scale=1 1 1
- link c1_lf: geometry collision mesh filename=../meshes/connect_coll.STL scale=1 1 1; visual mesh filename=../meshes/connect.STL scale=1 1 1
- link c1_lm: geometry collision mesh filename=../meshes/connect_coll.STL scale=1 1 1; visual mesh filename=../meshes/connect.STL scale=1 1 1
- link c1_lr: geometry collision mesh filename=../meshes/connect_coll.STL scale=1 1 1; visual mesh filename=../meshes/connect.STL scale=1 1 1
- link c1_rf: geometry collision mesh filename=../meshes/connect_coll.STL scale=1 1 1; visual mesh filename=../meshes/connect.STL scale=1 1 1
- link c1_rm: geometry collision mesh filename=../meshes/connect_coll.STL scale=1 1 1; visual mesh filename=../meshes/connect.STL scale=1 1 1
- link c1_rr: geometry collision mesh filename=../meshes/connect_coll.STL scale=1 1 1; visual mesh filename=../meshes/connect.STL scale=1 1 1
- link c2_lf: geometry collision mesh filename=../meshes/connect_coll.STL scale=1 1 1; visual mesh filename=../meshes/connect.STL scale=1 1 1
- link c2_lm: geometry collision mesh filename=../meshes/connect_coll.STL scale=1 1 1; visual mesh filename=../meshes/connect.STL scale=1 1 1
- link c2_lr: geometry collision mesh filename=../meshes/connect_coll.STL scale=1 1 1; visual mesh filename=../meshes/connect.STL scale=1 1 1
- link c2_rf: geometry collision mesh filename=../meshes/connect_coll.STL scale=1 1 1; visual mesh filename=../meshes/connect.STL scale=1 1 1
- link c2_rm: geometry collision mesh filename=../meshes/connect_coll.STL scale=1 1 1; visual mesh filename=../meshes/connect.STL scale=1 1 1
- link c2_rr: geometry collision mesh filename=../meshes/connect_coll.STL scale=1 1 1; visual mesh filename=../meshes/connect.STL scale=1 1 1
- link thigh_lf: geometry collision mesh filename=../meshes/thigh_l_coll.STL scale=1 1 1; visual mesh filename=../meshes/thigh_l.STL scale=1 1 1
- link thigh_lm: geometry collision mesh filename=../meshes/thigh_l_coll.STL scale=1 1 1; visual mesh filename=../meshes/thigh_l.STL scale=1 1 1
- link thigh_lr: geometry collision mesh filename=../meshes/thigh_l_coll.STL scale=1 1 1; visual mesh filename=../meshes/thigh_l.STL scale=1 1 1
- link thigh_rf: geometry collision mesh filename=../meshes/thigh_l_coll.STL scale=1 1 1; visual mesh filename=../meshes/thigh_l.STL scale=1 1 1
- link thigh_rm: geometry collision mesh filename=../meshes/thigh_l_coll.STL scale=1 1 1; visual mesh filename=../meshes/thigh_l.STL scale=1 1 1
- link thigh_rr: geometry collision mesh filename=../meshes/thigh_l_coll.STL scale=1 1 1; visual mesh filename=../meshes/thigh_l.STL scale=1 1 1
- link tibia_lf: geometry collision mesh filename=../meshes/tibia_l_coll.STL scale=1 1 1; visual mesh filename=../meshes/tibia_l.STL scale=1 1 1
- link tibia_lm: geometry collision mesh filename=../meshes/tibia_l_coll.STL scale=1 1 1; visual mesh filename=../meshes/tibia_l.STL scale=1 1 1
- link tibia_lr: geometry collision mesh filename=../meshes/tibia_l_coll.STL scale=1 1 1; visual mesh filename=../meshes/tibia_l.STL scale=1 1 1
- link tibia_rf: geometry collision mesh filename=../meshes/tibia_l_coll.STL scale=1 1 1; visual mesh filename=../meshes/tibia_l.STL scale=1 1 1
- link tibia_rm: geometry collision mesh filename=../meshes/tibia_l_coll.STL scale=1 1 1; visual mesh filename=../meshes/tibia_l.STL scale=1 1 1
- link tibia_rr: geometry collision mesh filename=../meshes/tibia_l_coll.STL scale=1 1 1; visual mesh filename=../meshes/tibia_l.STL scale=1 1 1

Commit message: Spatial Inertial Fails now

File: apps/models/urdf/phantomx.urdf (robot description, URDF)
Before this commit: robot PhantomX, 26 links, 25 joints
Links:
- link MP_BODY: geometry collision mesh filename=../meshes/collision/body_coll.obj scale=1 1 1; visual mesh filename=../meshes/body.STL scale=1 1 1
- link c1_lf: geometry collision mesh filename=../meshes/collision/connect_coll.obj scale=1 1 1; visual mesh filename=../meshes/connect.STL scale=1 1 1
- link c1_lm: geometry collision mesh filename=../meshes/collision/connect_coll.obj scale=1 1 1; visual mesh filename=../meshes/connect.STL scale=1 1 1
- link c1_lr: geometry collision mesh filename=../meshes/collision/connect_coll.obj scale=1 1 1; visual mesh filename=../meshes/connect.STL scale=1 1 1
- link c1_rf: geometry collision mesh filename=../meshes/collision/connect_coll.obj scale=1 1 1; visual mesh filename=../meshes/connect.STL scale=1 1 1
- link c1_rm: geometry collision mesh filename=../meshes/collision/connect_coll.obj scale=1 1 1; visual mesh filename=../meshes/connect.STL scale=1 1 1
- link c1_rr: geometry collision mesh filename=../meshes/collision/connect_coll.obj scale=1 1 1; visual mesh filename=../meshes/connect.STL scale=1 1 1
- link c2_lf: geometry collision mesh filename=../meshes/collision/connect_coll.obj scale=1 1 1; visual mesh filename=../meshes/connect.STL scale=1 1 1
- link c2_lm: geometry collision mesh filename=../meshes/collision/connect_coll.obj scale=1 1 1; visual mesh filename=../meshes/connect.STL scale=1 1 1
- link c2_lr: geometry collision mesh filename=../meshes/collision/connect_coll.obj scale=1 1 1; visual mesh filename=../meshes/connect.STL scale=1 1 1
- link c2_rf: geometry collision mesh filename=../meshes/collision/connect_coll.obj scale=1 1 1; visual mesh filename=../meshes/connect.STL scale=1 1 1
- link c2_rm: geometry collision mesh filename=../meshes/collision/connect_coll.obj scale=1 1 1; visual mesh filename=../meshes/connect.STL scale=1 1 1
- link c2_rr: geometry collision mesh filename=../meshes/collision/connect_coll.obj scale=1 1 1; visual mesh filename=../meshes/connect.STL scale=1 1 1
- link thigh_lf: geometry collision mesh filename=../meshes/collision/thigh_l_coll.obj scale=1 1 1; visual mesh filename=../meshes/thigh_l.STL scale=1 1 1
- link thigh_lm: geometry collision mesh filename=../meshes/collision/thigh_l_coll.obj scale=1 1 1; visual mesh filename=../meshes/thigh_l.STL scale=1 1 1
- link thigh_lr: geometry collision mesh filename=../meshes/collision/thigh_l_coll.obj scale=1 1 1; visual mesh filename=../meshes/thigh_l.STL scale=1 1 1
- link thigh_rf: geometry collision mesh filename=../meshes/collision/thigh_l_coll.obj scale=1 1 1; visual mesh filename=../meshes/thigh_l.STL scale=1 1 1
- link thigh_rm: geometry collision mesh filename=../meshes/collision/thigh_l_coll.obj scale=1 1 1; visual mesh filename=../meshes/thigh_l.STL scale=1 1 1
- link thigh_rr: geometry collision mesh filename=../meshes/collision/thigh_l_coll.obj scale=1 1 1; visual mesh filename=../meshes/thigh_l.STL scale=1 1 1
- link tibia_lf: geometry collision mesh filename=../meshes/collision/tibia_l_coll.obj scale=1 1 1; visual mesh filename=../meshes/tibia_l.STL scale=1 1 1
- link tibia_lm: geometry collision mesh filename=../meshes/collision/tibia_l_coll.obj scale=1 1 1; visual mesh filename=../meshes/tibia_l.STL scale=1 1 1
- link tibia_lr: geometry collision mesh filename=../meshes/collision/tibia_l_coll.obj scale=1 1 1; visual mesh filename=../meshes/tibia_l.STL scale=1 1 1
- link tibia_rf: geometry collision mesh filename=../meshes/collision/tibia_l_coll.obj scale=1 1 1; visual mesh filename=../meshes/tibia_l.STL scale=1 1 1
- link tibia_rm: geometry collision mesh filename=../meshes/collision/tibia_l_coll.obj scale=1 1 1; visual mesh filename=../meshes/tibia_l.STL scale=1 1 1
- link tibia_rr: geometry collision mesh filename=../meshes/collision/tibia_l_coll.obj scale=1 1 1; visual mesh filename=../meshes/tibia_l.STL scale=1 1 1
